File: Shimonso-IoT-Type-R.kicad_pcb (KiCad board)
At the start: 4 copper layers, 85 x 54 mm, 111 parts, among them CON1 96Boards_HS_connector, CON2 96Boards_LS_connector, P2 USB_OTG, P4 CONN_01X15, P5 CONN_01X15, Q1 S8050, SW1 RST, U1 FT230X, U10 bh1745nuc, U11 BU9873, U12 ADS1115, U13 BD1020HFV, U14 ML8511A, U15 PCA9306DC1, U16 PCA9306DC1, U17 MC-306_32.768K-E3, U18 SN74AVC4T245, U2 BD33GC0WEFJ, U3 PCA9306DC1, U4 BD18GC0WEFJ, U5 bd7411g, U6 kx022-1020, U7 bm1383glv, U8 bm1422gmv, U9 rpr-0521rs

Commit message: modified
Parts:
- removed P2: USB_OTG, droneworks:10118194-0001LF
- removed P4, P5: CONN_01X15, droneworks:1-84952-5
- added CON3: microUSB_CONSOLE, droneworks:10118194-0001LF, F.Cu at (63.1, 150.0)
- added CON4: CONN_01X15, droneworks:1-84952-5, F.Cu at (96.3, 143.0)
- added CON5: CONN_01X15, droneworks:1-84952-5, F.Cu at (122.3, 143.0)
- added TH2: TH, Pin_Headers:Pin_Header_Straight_1x01, F.Cu at (52.2, 148.1)
- added TH3: TH, Pin_Headers:Pin_Header_Straight_1x01, F.Cu at (126.1, 99.9)
- added TH4: TH, Pin_Headers:Pin_Header_Straight_1x01, F.Cu at (99.4, 104.2)
- added TH5: TH, Pin_Headers:Pin_Header_Straight_1x01, F.Cu at (102.9, 104.2)
- added TH6: TH, Pin_Headers:Pin_Header_Straight_1x01, F.Cu at (106.4, 104.2)
- CB12, CB13, CB14: value 1.0uF -> 104
- CB16: value 10uF -> 104
- CB19: value 104 -> 1.0uF
- CB20: value 10uF -> 1.0uF
- CB21: value 1nF -> 1.0uF
- CB23, CB24: value 104 -> 0
- CB25, CB30: value 104 -> 10uF
- CB27, CB28: value 0 -> 104
- CB31: value 104 -> 1nF
- D1: moved to B.Cu
- LED5, LED6: moved to F.Cu
- R1, R2: value 22 -> 220
- R10, R26, R9: value 4.7k -> 2.2k
- R11: value 1k -> 2.2k
- R12: value 2.2k -> 10K
- R13, R14: value 2.2k -> 220
- R16: value 2.2k -> 220; moved to F.Cu
- R17, R18: value 200k -> 220; moved to F.Cu
- R19: value 2.2k -> 160; moved to F.Cu
- R20, R21: value 2.2k -> 200k
- R22: value 2.2k -> 18k; moved to F.Cu
- R23: value 18k -> 2.2k
- R24: value 10k -> 2.2k
- R25: value 200k -> 10k; moved to F.Cu
- R27: value 220 -> 2.2k
- R28: value 220 -> 200k
- R29: value 390 -> 2.2k
- R3: value 10K -> 390
- R30: value 620 -> 2.2k
- R31, R33: value 220 -> 4.7k
- R32: value 220 -> 1k
- R34: value 160 -> 4.7k
- R4: value 220 -> 620; moved to F.Cu
- R5: value 220 -> 22
- R6: value 2.2k -> 22
- TH1: footprint droneworks:B3U-1000P -> Pin_Headers:Pin_Header_Straight_1x01; moved to F.Cu
- U10: value bh1745nuc -> PCA9306DC1; footprint rohm:BH1745NUC -> droneworks:PCA9306DC1
- U11: value BU9873 -> bm1422gmv; footprint rohm:BU9873F-GTE2 -> rohm:BM1422GMV
- U12: value ADS1115 -> BU9873; footprint droneworks:ADS1115 -> rohm:BU9873F-GTE2
- U13: value BD1020HFV -> rpr-0521rs; footprint rohm:BD1020HFV -> rohm:RPR-0521RS
- U14: value ML8511A -> bh1745nuc; footprint rohm:ML8511A -> rohm:BH1745NUC
- U15: value PCA9306DC1 -> ADS1115; footprint droneworks:PCA9306DC1 -> droneworks:ADS1115
- U16: value PCA9306DC1 -> MC-306_32.768K-E3; footprint droneworks:PCA9306DC1 -> droneworks:MC-306
- U17: value MC-306_32.768K-E3 -> BD1020HFV; footprint droneworks:MC-306 -> rohm:BD1020HFV
- U18: value SN74AVC4T245 -> ML8511A; footprint droneworks:SN74AVC4T245PWT -> rohm:ML8511A
- U3: value PCA9306DC1 -> BD18GC0WEFJ; footprint droneworks:PCA9306DC1 -> rohm:BDxxGC0WEFJ
- U4: value BD18GC0WEFJ -> SN74AVC4T245; footprint rohm:BDxxGC0WEFJ -> droneworks:SN74AVC4T245PWT
- U5: value bd7411g -> PCA9306DC1; footprint rohm:BD7411G -> droneworks:PCA9306DC1
- U6: value kx022-1020 -> PCA9306DC1; footprint rohm:KX022-1020 -> droneworks:PCA9306DC1
- U7: value bm1383glv -> bd7411g; footprint rohm:BM1383GLV -> rohm:BD7411G
- U8: value bm1422gmv -> kx022-1020; footprint rohm:BM1422GMV -> rohm:KX022-1020
- U9: value rpr-0521rs -> bm1383glv; footprint rohm:RPR-0521RS -> rohm:BM1383GLV
- moved CB2 138.1 mm to (54.2, 135.4), turned to 180 degrees
- moved CB24 133.1 mm to (55.4, 108.2), turned to 180 degrees
- moved CB28 131.1 mm to (56.8, 115.8), turned to 180 degrees
- moved LED6 130.0 mm to (74.6, 143.6)
- moved CB23 129.5 mm to (55.4, 105.4), turned to 180 degrees
- moved LED5 126.4 mm to (74.6, 140.9)
- moved CB1 124.9 mm to (51.9, 144.1), turned to 270 degrees
- moved R14 122.2 mm to (64.0, 135.8), turned to 270 degrees
- moved CB17 120.9 mm to (75.5, 107.7)
- moved R6 115.3 mm to (55.5, 143.2), turned to 180 degrees
- moved R28 114.3 mm to (71.7, 107.2)
- moved CB31 112.6 mm to (85.7, 129.7), turned to 270 degrees
- moved CC1 105.6 mm to (56.8, 146.8), turned to 270 degrees
- moved LED4 104.4 mm to (122.1, 99.7), turned to 90 degrees
- moved R8 102.1 mm to (102.2, 133.1)
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Connections:
- CB11 pad 1: /1V8 -> /3V3
- CB12 pad 1: /1V8 -> Net-(CB12-Pad1)
- CB14 pad 1: Net-(CB14-Pad1) -> /3V3
- CB15 pad 1: /3V3 -> /1V8
- CB17 pad 1: /3V3 -> Net-(CB17-Pad1)
- CB18 pad 1: /3V3 -> /1V8
- CB19 pad 1: /3V3 -> /1V8
- CB2 pad 1: /3V3 -> Net-(CB2-Pad1)
- CB20 pad 1: /3V3 -> Net-(CB20-Pad1)
- CB23 pad 1: /1V8 -> Net-(CB23-Pad1)
- CB24 pad 1: /1V8 -> Net-(CB24-Pad1)
- CB25 pad 1: Net-(CB25-Pad1) -> /3V3
- CB26 pad 1: Net-(CB26-Pad1) -> /3V3
- CB27 pad 1: Net-(CB27-Pad1) -> /3V3
- CB29 pad 1: Net-(CB29-Pad1) -> /3V3
- CB30 pad 1: /1V8 -> /3V3
- CB31 pad 1: /3V3 -> Net-(CB31-Pad1)
- CB6 pad 1: /3V3 -> /1V8
- CB9 pad 1: Net-(CB9-Pad1) -> /1V8
- CE8 pad 1: Net-(CB29-Pad1) -> Net-(CB28-Pad1)
- D1 pad 1: Net-(CB29-Pad1) -> Net-(CB28-Pad1)
- R1 pad 1: Net-(R1-Pad1) -> Net-(Q1-Pad2)
- R1 pad 2: /USBDM -> Net-(CON2-Pad27)
- R10 pad 2: /BH1745NUC_INT -> /ISP0_SDA
- R11 pad 1: Net-(C1-Pad1) -> /1V8
- R11 pad 2: Net-(CB29-Pad1) -> Net-(R11-Pad2)
- R12 pad 1: /1V8 -> GND
- R12 pad 2: /ISP1_SDA -> Net-(R12-Pad2)
- R13 pad 1: /1V8 -> /PMU_PWRON_N
- R13 pad 2: /ISP0_SCL -> Net-(R13-Pad2)
- R14 pad 1: /1V8 -> /EXP_RSTOUT_N
- R14 pad 2: /ISP0_SDA -> Net-(R14-Pad2)
- R16 pad 1: /1V8 -> /3V3
- R16 pad 2: Net-(R16-Pad2) -> Net-(LED5-Pad2)
- R17 pad 2: Net-(CB25-Pad1) -> Net-(LED6-Pad2)
- R18 pad 2: Net-(CB26-Pad1) -> Net-(LED3-Pad2)
- R19 pad 1: /3V3 -> /1V8
- R19 pad 2: /ISP1_SCL_3V3 -> Net-(LED4-Pad2)
- R2 pad 1: Net-(R2-Pad1) -> GND
- R2 pad 2: /USBDP -> Net-(Q1-Pad2)
- R20 pad 2: /ISP1_SDA_3V3 -> Net-(CB12-Pad1)
- R21 pad 2: /ISP0_SCL_3V3 -> Net-(CB13-Pad1)
- R22 pad 1: /3V3 -> /BD7411G_OUT_1V8
- R22 pad 2: /ISP0_SDA_3V3 -> /BD7411G_OUT_5V
- R23 pad 1: /BD7411G_OUT_1V8 -> /3V3
- R23 pad 2: /BD7411G_OUT_5V -> /ISP1_SCL_3V3
- R24 pad 1: /BD7411G_OUT_1V8 -> /3V3
- R24 pad 2: GND -> /ISP1_SDA_3V3
- R25 pad 1: /3V3 -> /BD7411G_OUT_1V8
- R25 pad 2: Net-(CB9-Pad1) -> GND
- R26 pad 1: /1V8 -> /3V3
- R26 pad 2: /BM1383GLV_INT -> /ISP0_SCL_3V3
- R27 pad 1: Net-(Q1-Pad2) -> /3V3
- R27 pad 2: Net-(CON2-Pad27) -> /ISP0_SDA_3V3
- R28 pad 1: GND -> /3V3
- R28 pad 2: Net-(Q1-Pad2) -> Net-(CB17-Pad1)
- R29 pad 1: /5V -> /3V3
- R29 pad 2: Net-(LED1-Pad2) -> /I2C0_SCL_3V3
- R3 pad 1: GND -> /5V
- R3 pad 2: Net-(R3-Pad2) -> Net-(LED1-Pad2)
- R30 pad 1: /5V -> /3V3
- R30 pad 2: Net-(LED2-Pad2) -> /I2C0_SDA_3V3
- R31 pad 1: /3V3 -> /1V8
- R31 pad 2: Net-(LED5-Pad2) -> /BM1383GLV_INT
- R32 pad 1: /3V3 -> Net-(C1-Pad1)
- R32 pad 2: Net-(LED6-Pad2) -> Net-(CB28-Pad1)
- R33 pad 1: /3V3 -> /1V8
- R33 pad 2: Net-(LED3-Pad2) -> /RPR-0521RS_INT
- R34 pad 2: Net-(LED4-Pad2) -> /BH1745NUC_INT
- R4 pad 1: /PMU_PWRON_N -> /5V
- R4 pad 2: Net-(R4-Pad2) -> Net-(LED2-Pad2)
- R5 pad 1: /EXP_RSTOUT_N -> Net-(R5-Pad1)
- R5 pad 2: Net-(R5-Pad2) -> /USBDM
- R6 pad 1: /3V3 -> Net-(R6-Pad1)
- R6 pad 2: /I2C0_SCL_3V3 -> /USBDP
- R7 pad 1: /3V3 -> /1V8
- R7 pad 2: /I2C0_SDA_3V3 -> /ISP1_SCL
- R8 pad 2: /ISP1_SCL -> /ISP1_SDA
- R9 pad 2: /RPR-0521RS_INT -> /ISP0_SCL
- U1 pad 10: /3V3 -> Net-(CB2-Pad1)
- U1 pad 11: /3V3 -> Net-(CB2-Pad1)
- U1 pad 16: Net-(R5-Pad2) -> Net-(R14-Pad2)
- U1 pad 3: /3V3 -> /1V8
- U1 pad 6: Net-(R3-Pad2) -> Net-(R12-Pad2)
- U1 pad 7: Net-(R4-Pad2) -> Net-(R13-Pad2)
- U1 pad 8: Net-(R2-Pad1) -> Net-(R6-Pad1)
- U1 pad 9: Net-(R1-Pad1) -> Net-(R5-Pad1)
- U10 pad 1: /3V3 -> GND
- U10 pad 2: /3V3 -> /1V8
- U10 pad 3: GND -> /I2C0_SCL
- U10 pad 4: GND -> /I2C0_SDA
- U10 pad 5: /I2C0_SCL_3V3 -> /I2C0_SDA_3V3
- U10 pad 6: /I2C0_SDA_3V3 -> /I2C0_SCL_3V3
- U10 pad 7: /BH1745NUC_INT -> Net-(CB17-Pad1)
- U10 pad 8: Net-(U10-Pad8) -> Net-(CB17-Pad1)
- U11 pad 1: Net-(U11-Pad1) -> /1V8
- U11 pad 2: /I2C0_SCL_3V3 -> GND
- U11 pad 3: /I2C0_SDA_3V3 -> Net-(CB21-Pad1)
- U11 pad 4: GND -> Net-(U11-Pad4)
- U11 pad 5: Net-(U11-Pad5) -> /I2C0_SDA
- U11 pad 6: Net-(CB27-Pad1) -> Net-(U11-Pad6)
- U11 pad 7: Net-(CB28-Pad1) -> /I2C0_SCL
- U11 pad 8: Net-(CB29-Pad1) -> /BM1422GMV_DRDY
- U12 pad 1: /3V3 -> Net-(U12-Pad1)
- U12 pad 2: Net-(U12-Pad2) -> /I2C0_SCL_3V3
- U12 pad 3: GND -> /I2C0_SDA_3V3
- U12 pad 4: Net-(U12-Pad4) -> GND
- U12 pad 6: Net-(U12-Pad6) -> Net-(CB23-Pad1)
- U12 pad 7: Net-(U12-Pad7) -> Net-(CB24-Pad1)
- U12 pad 8: /3V3 -> Net-(CB28-Pad1)
- U13 pad 1: Net-(U13-Pad1) -> /3V3
- U13 pad 2: Net-(PAD1-Pad1) -> /I2C0_SCL_3V3
- U13 pad 3: Net-(U12-Pad4) -> GND
- U13 pad 5: GND -> Net-(U13-Pad5)
- U14 pad 1: Net-(U14-Pad1) -> /3V3
- U14 pad 2: Net-(U14-Pad2) -> /3V3
- U14 pad 3: Net-(U14-Pad3) -> GND
- U14 pad 4: /3V3 -> GND
- U14 pad 5: GND -> /I2C0_SCL_3V3
- U14 pad 6: Net-(U14-Pad6) -> /I2C0_SDA_3V3
- U14 pad 7: /3V3 -> /BH1745NUC_INT
- U14 pad 8: Net-(U12-Pad5) -> Net-(U14-Pad8)
- U15 pad 1: GND -> /3V3
- U15 pad 2: /1V8 -> Net-(U15-Pad2)
- U15 pad 3: /ISP0_SCL -> GND
- U15 pad 4: /ISP0_SDA -> Net-(U15-Pad4)
- U15 pad 5: /ISP0_SDA_3V3 -> Net-(U15-Pad5)
- U15 pad 6: /ISP0_SCL_3V3 -> Net-(U15-Pad6)
- U15 pad 7: Net-(CB25-Pad1) -> Net-(U15-Pad7)
- U15 pad 8: Net-(CB25-Pad1) -> /3V3
- U16 pad 1: GND -> Net-(CB24-Pad1)
- U16 pad 2: /1V8 -> Net-(U16-Pad2)
- U16 pad 3: /ISP1_SCL -> Net-(U16-Pad3)
- U16 pad 4: /ISP1_SDA -> Net-(CB23-Pad1)
- U17 pad 1: Net-(CB28-Pad1) -> Net-(U17-Pad1)
- U17 pad 2: Net-(U17-Pad2) -> Net-(PAD1-Pad1)
- U17 pad 3: Net-(U17-Pad3) -> Net-(U15-Pad4)
- U17 pad 4: Net-(CB27-Pad1) -> /3V3
- U18 pad 1: /1V8 -> Net-(U18-Pad1)
- U18 pad 10: /CAM2_CLK_3V3 -> Net-(CB31-Pad1)
- U18 pad 11: /CAM1_CLK_3V3 -> Net-(U18-Pad11)
- U18 pad 12: /CAM2_GPIO_3V3 -> Net-(U18-Pad12)
- U18 pad 2: Net-(R15-Pad2) -> Net-(U18-Pad2)
- U18 pad 3: Net-(R16-Pad2) -> Net-(U18-Pad3)
- U18 pad 4: /CAM1_GPIO -> /3V3
- U18 pad 5: /CAM2_GPIO -> GND
- U18 pad 6: /CAM1_CLK -> Net-(U18-Pad6)
- U18 pad 7: /CAM2_CLK -> /3V3
- U18 pad 8: GND -> Net-(U15-Pad5)
- U18 pad 9: GND -> Net-(U18-Pad9)
- U3 pad 1: GND -> /1V8
- U3 pad 3: /I2C0_SCL -> GND
- U3 pad 4: /I2C0_SDA -> Net-(U3-Pad4)
- U3 pad 5: /I2C0_SDA_3V3 -> /5V
- U3 pad 6: /I2C0_SCL_3V3 -> Net-(U3-Pad6)
- U3 pad 7: Net-(CB9-Pad1) -> Net-(U3-Pad7)
- U3 pad 8: Net-(CB9-Pad1) -> /5V
- U4 pad 2: /1V8 -> Net-(R11-Pad2)
- U4 pad 3: GND -> Net-(R15-Pad2)
- U4 pad 4: Net-(U4-Pad4) -> /CAM1_GPIO
- U4 pad 5: /5V -> /CAM2_GPIO
- U4 pad 6: Net-(U4-Pad6) -> /CAM1_CLK
- U4 pad 7: Net-(U4-Pad7) -> /CAM2_CLK
- U4 pad 8: /5V -> GND
- U5 pad 1: Net-(U5-Pad1) -> GND
- U5 pad 2: GND -> /1V8
- U5 pad 3: Net-(U5-Pad3) -> /ISP0_SCL
- U5 pad 4: /BD7411G_OUT_5V -> /ISP0_SDA
- U5 pad 5: /5V -> /ISP0_SDA_3V3
- U6 pad 2: /I2C0_SDA -> /1V8
- U6 pad 3: /1V8 -> /ISP1_SCL
- U6 pad 4: GND -> /ISP1_SDA
- U6 pad 5: /KX022-1020_INT1 -> /ISP1_SDA_3V3
- U6 pad 6: Net-(U6-Pad6) -> /ISP1_SCL_3V3
- U6 pad 7: /1V8 -> Net-(CB13-Pad1)
- U6 pad 8: GND -> Net-(CB13-Pad1)
- U7 pad 1: Net-(CB13-Pad1) -> Net-(U7-Pad1)
- U7 pad 2: /1V8 -> GND
- U7 pad 3: GND -> Net-(U7-Pad3)
- U7 pad 4: Net-(U7-Pad4) -> /BD7411G_OUT_5V
- U7 pad 5: Net-(U7-Pad4) -> /5V
- U8 pad 1: /1V8 -> GND
- U8 pad 2: GND -> /I2C0_SDA
- U8 pad 3: Net-(CB14-Pad1) -> /1V8
- U8 pad 4: Net-(U8-Pad4) -> GND
- U8 pad 5: /I2C0_SDA -> /KX022-1020_INT1
- U8 pad 7: /I2C0_SCL -> /1V8
- U8 pad 8: /BM1422GMV_DRDY -> GND
- U9 pad 1: /3V3 -> Net-(CB20-Pad1)
- U9 pad 2: /I2C0_SCL_3V3 -> /1V8
- U9 pad 4: /3V3 -> Net-(U9-Pad4)
- U9 pad 5: Net-(U9-Pad5) -> Net-(U9-Pad4)
- U9 pad 6: Net-(U9-Pad5) -> GND
- U9 pad 7: /RPR-0521RS_INT -> Net-(U9-Pad7)
- U9 pad 8: /I2C0_SDA_3V3 -> Net-(U9-Pad8)
Other:
- outline, holes or cut-outs redrawn

Commit message: modified
Parts:
- R18, R19, R27, R4: moved to B.Cu
- R23, R26: moved to F.Cu
- moved CB7 57.1 mm to (98.8, 135.5), turned to 180 degrees
- moved CB11 57.1 mm to (114.3, 119.9)
- moved CB5 55.1 mm to (108.5, 123.2)
- moved R26 49.7 mm to (99.1, 140.2)
- moved R20 46.7 mm to (107.0, 139.6), turned to 180 degrees
- moved CB16 43.5 mm to (106.5, 142.3)
- moved CB10 43.4 mm to (114.3, 122.8)
- moved CB13 32.4 mm to (123.7, 136.5), turned to 180 degrees
- moved R23 32.2 mm to (125.8, 140.7)
- moved CB14 30.4 mm to (132.5, 142.3)
- moved R7 29.1 mm to (126.6, 131.4), turned to 270 degrees
- moved CB6 29.1 mm to (132.9, 134.8)
- moved U6 28.6 mm to (127.9, 137.1), turned to 180 degrees
- moved CON4 26.0 mm to (122.3, 143.0)
- moved CON5 25.8 mm to (96.5, 143.0)
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
Commit message: placement modified
Parts:
- CB26, R22, R25, R28, R29: moved to B.Cu
- R32: moved to F.Cu
- moved CB26 98.3 mm to (66.7, 120.1), turned to 270 degrees
- moved R34 94.6 mm to (66.4, 117.3)
- moved CB25 89.4 mm to (73.9, 112.8)
- moved CB27 84.7 mm to (65.0, 112.2), turned to 180 degrees
- moved CB15 80.0 mm to (78.2, 107.3)
- moved CB30 77.4 mm to (80.2, 128.1)
- moved R33 77.0 mm to (73.9, 115.4), turned to 180 degrees
- moved CB22 75.4 mm to (82.7, 118.4)
- moved R2 68.8 mm to (90.2, 103.9), turned to 180 degrees
- moved CB20 67.8 mm to (94.6, 117.5)
- moved CB29 66.8 mm to (65.0, 114.6), turned to 180 degrees
- moved CB32 66.6 mm to (91.8, 123.0)
- moved CB8 61.7 mm to (125.4, 109.4), turned to 180 degrees
- moved R31 61.0 mm to (94.7, 114.9)
- moved CB18 60.8 mm to (108.8, 110.1)
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
Commit message: modified
Routing:
- net GND: track 0.00 -> 569.9 mm, vias 0 -> 7
- net /3V3: track 0.00 -> 255.4 mm, vias 0 -> 12
- net /1V8: track 0.00 -> 212.8 mm, vias 0 -> 4
- net /5V: track 0.00 -> 85.1 mm, vias 0 -> 3
- net /EXP_RSTOUT_N: track 0.00 -> 59.6 mm, vias 0 -> 1
- net /BM1383GLV_INT: track 0.00 -> 54.5 mm, vias 0 -> 3
- net /CSI1_DATA0_N: track 0.00 -> 53.2 mm, vias 0 -> 1
- net /CSI1_DATA0_P: track 0.00 -> 51.8 mm, vias 0 -> 1
- net /PMU_PWRON_N: track 0.00 -> 48.3 mm
- net /CAM1_GPIO: track 0.00 -> 48.2 mm, vias 0 -> 1
- net /CSI1_DATA1_P: track 0.00 -> 47.8 mm, vias 0 -> 1
- net /CAM2_GPIO: track 0.00 -> 46.8 mm, vias 0 -> 2
- net /CSI1_DATA1_N: track 0.00 -> 45.4 mm, vias 0 -> 1
- net /UART3_TX: track 0.00 -> 45.1 mm, vias 0 -> 1
- net /UART3_RX: track 0.00 -> 45.0 mm, vias 0 -> 1
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
Commit message: modified
Parts:
- CB1, R12: moved to F.Cu
- LED1, LED2, LED3, LED4, LED5, LED6: footprint LEDs:LED_0603 -> droneworks:LED_1608mm
- TH1, TH2, TH3, TH4, TH5, TH6: footprint Pin_Headers:Pin_Header_Straight_1x01 -> droneworks:TH
- moved CB2 18.7 mm to (71.9, 141.4), turned to 90 degrees
- moved R13 15.7 mm to (53.4, 141.8), turned to 0 degrees
- moved R12 15.5 mm to (51.7, 138.7), turned to 270 degrees
- moved SW1 4.61 mm to (64.9, 132.3)
- moved CC2 2.06 mm to (69.6, 146.9)
- moved R6 1.77 mm to (56.8, 144.4), turned to 270 degrees
- moved TH1 1.50 mm to (54.5, 138.8)
- moved R5 1.34 mm to (69.6, 144.0), turned to 270 degrees
- moved R14 1.03 mm to (64.9, 136.3)
- moved CB1 1.03 mm to (52.8, 143.6)
- moved R17 0.80 mm to (78.5, 148.6)
- moved LED6 0.60 mm to (74.6, 148.6)
- moved CB30 0.50 mm to (80.2, 128.6)
- moved CC1 0.50 mm to (56.8, 147.3)
- moved LED5 0.20 mm to (74.6, 145.3)
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Routing:
- net GND: track 569.9 -> 486.5 mm, vias 7 -> 19
- net /1V8: track 212.8 -> 181.8 mm
- net /3V3: track 255.4 -> 229.0 mm, vias 12 -> 13
- net Net-(R13-Pad2): track 26.2 -> 7.28 mm
- net /5V: track 85.1 -> 70.1 mm, vias 3 -> 5
- net Net-(CB2-Pad1): track 24.9 -> 11.5 mm
- net /CSI1_DATA1_P: track 47.8 -> 38.4 mm, vias 1 -> 0
- net /PMU_PWRON_N: track 48.3 -> 56.9 mm
- net /+5F: track 33.7 -> 25.2 mm, vias 3 -> 2
- net /CSI1_CLK_P: track 40.3 -> 32.3 mm, vias 3 -> 2
- net Net-(R12-Pad2): track 18.3 -> 10.3 mm, vias 1 -> 0
- net /USBDM: track 14.0 -> 9.94 mm
- net Net-(CB23-Pad1): track 7.34 -> 3.73 mm, vias 1 -> 0
- net /USBDP: track 11.8 -> 8.60 mm
- net Net-(CB24-Pad1): track 7.34 -> 4.16 mm, vias 1 -> 0
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- added copper zone on In1.Cu, net GND
Other:
- net class 5V added: clearance 0.25, trace_width 0.35, via_dia 0.6, via_drill 0.4
- net class GND added: clearance 0.25, trace_width 0.35, via_dia 0.6, via_drill 0.4

Commit message: modified
Parts:
- R26: moved to B.Cu
- moved R26 5.97 mm to (100.5, 146.0)
- moved R27 0.22 mm to (103.5, 146.0)
Routing:
- net GND: track 486.5 -> 433.5 mm, vias 19 -> 36
- net /3V3: track 229.0 -> 202.8 mm, vias 13 -> 11
- net /1V8: track 181.8 -> 164.0 mm
- net /CSI1_DATA1_P: track 38.4 -> 48.0 mm, vias 0 -> 1
- net /CAM1_CLK: track 42.3 -> 35.0 mm
- net /CSI0_DATA1_P: track 32.0 -> 26.0 mm
- net /CSI0_DATA0_N: track 28.5 -> 22.6 mm
- net /CSI0_DATA1_N: track 29.7 -> 24.0 mm
- net /CAM1_CLK_3V3: track 26.1 -> 20.4 mm
- net /CSI0_DATA0_P: track 32.4 -> 27.0 mm, vias 3 -> 1
- net /CAM1_GPIO_3V3: track 27.1 -> 22.1 mm
- net /CSI0_CLK_N: track 38.2 -> 35.0 mm
- net /CSI1_CLK_P: track 32.3 -> 29.3 mm
- net /CSI1_DATA0_P: track 51.8 -> 53.5 mm
- net /I2C0_SDA: track 0.00 -> 1.25 mm
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Other:
- net class 5V: trace_width 0.35 -> 0.25
- net class ISP0_SCL_3V3 added: clearance 0.2, trace_width 0.2, via_dia 0.6, via_drill 0.4
- rule trace_min: 0.25 -> 0.2

Commit message: modified
Parts:
- CB25, R23: moved to B.Cu
- CB28, CB7, D1, R10, R3, R9: moved to F.Cu
- moved CB7 8.01 mm to (105.8, 139.3), turned to 0 degrees
- moved R9 7.62 mm to (97.6, 138.0), turned to 90 degrees
- moved R34 6.30 mm to (72.7, 117.3), turned to 270 degrees
- moved R24 5.72 mm to (128.4, 140.4)
- moved R27 5.50 mm to (103.5, 140.5)
- moved R23 5.39 mm to (128.6, 145.3), turned to 180 degrees
- moved R33 4.83 mm to (77.0, 111.7), turned to 270 degrees
- moved R10 4.67 mm to (99.7, 136.9), turned to 90 degrees
- moved R26 2.11 mm to (102.6, 145.8), turned to 180 degrees
- moved R22 1.40 mm to (95.7, 107.4)
- moved R25 1.38 mm to (92.7, 107.4)
- moved R3 1.25 mm to (83.4, 104.5), turned to 270 degrees
- moved R31 1.22 mm to (93.7, 114.2), turned to 270 degrees
- moved LED1 1.22 mm to (83.4, 107.5), turned to 90 degrees
- moved C1 1.12 mm to (59.0, 122.7)
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Routing:
- net GND: track 433.5 -> 300.4 mm, vias 36 -> 53
- net /3V3: track 202.8 -> 153.7 mm, vias 11 -> 20
- net /1V8: track 164.0 -> 212.4 mm, vias 4 -> 14
- net /I2C0_SDA_3V3: track 0.00 -> 38.3 mm
- net /I2C0_SCL: track 23.2 -> 46.6 mm
- net /I2C0_SCL_3V3: track 11.7 -> 30.6 mm, vias 2 -> 1
- net /CSI1_DATA0_N: track 54.4 -> 38.2 mm
- net /5V: track 70.1 -> 83.7 mm
- net /CSI1_DATA0_P: track 53.5 -> 41.4 mm
- net /CSI1_CLK_P: track 29.3 -> 41.0 mm, vias 2 -> 3
- net Net-(CB28-Pad1): track 22.1 -> 15.7 mm, vias 1 -> 0
- net /ISP1_SDA: track 41.3 -> 47.3 mm
- net /I2C0_SDA: track 1.25 -> 6.27 mm, vias 0 -> 1
- net /ISP0_SCL_3V3: track 3.62 -> 8.62 mm
- net /ISP1_SCL: track 45.0 -> 49.6 mm, vias 2 -> 3
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- added copper zone on In2.Cu, net /3V3
Other:
- net class 0.15 added: clearance 0.15, trace_width 0.15, via_dia 0.6, via_drill 0.4
- net class 0.2 added: clearance 0.2, trace_width 0.25, via_dia 0.6, via_drill 0.4
- net class 1V8 added: clearance 0.4, trace_width 0.4, via_dia 0.6, via_drill 0.4
- net class 3V5 added: clearance 0.25, trace_width 0.35, via_dia 0.6, via_drill 0.4
- net class ISP0_SCL_3V3 removed
- net class SCL_SDA added: clearance 0.2, trace_width 0.2, via_dia 0.6, via_drill 0.4
- net class SCL_SDA_3V3 added: clearance 0.15, trace_width 0.15, via_dia 0.6, via_drill 0.4
- rule trace_min: 0.2 -> 0.15

Commit message: modified
Routing:
- net /I2C0_SDA: track 6.27 -> 50.5 mm, vias 1 -> 4
- net GND: track 300.4 -> 338.5 mm, vias 53 -> 61
- net /3V3: track 153.7 -> 116.3 mm, vias 20 -> 26
- net /1V8: track 212.4 -> 220.8 mm, vias 14 -> 16
- net Net-(U15-Pad5): track 0.00 -> 7.59 mm, vias 0 -> 2
- net Net-(U9-Pad4): track 1.86 -> 0.59 mm
- net Net-(CB17-Pad1): track 4.88 -> 5.38 mm
- net (no net): track 0.47 -> 0.07 mm, vias 1 -> 0
